File: eagle/emilyCircuit/emilyBoard.sch (EAGLE design)
At the start: 12 parts

Commit message: Updated EMILY PCB files with labels. Complies with OSHPark DRGs and Eagle ERGs.
Changed lines of the file:
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@@
 <wire x1="93.98" y1="40.64" x2="99.06" y2="40.64" width="0.1524" layer="91"/>
 <label x="99.06" y="40.64" size="1.778" layer="95"/>
+<junction x="93.98" y="40.64"/>
 </segment>
 <segment>
